Commit message: Relative path, velocity limits and inertia

File: Simulation/Button/Button_Assembly.urdf (robot description, URDF)
Before this commit: robot Button_Assembly, 3 links, 2 joints
Links:
- link World: mass None -> 0.1412
- link button_pivot: mass None -> 0.0377
- link lid_pivot: mass None -> 0.0824
Joints:
- joint PrismaticJoint: limit lower=-0.01 upper=0. effort=10000000. velocity=0. -> lower=-0.01 upper=0. effort=100.0 velocity=1.0
- joint RevoluteJoint: limit lower=-1.5707963 upper=0.6981317 effort=0. velocity=0. -> lower=-1.5707963 upper=0.6981317 effort=100.0 velocity=10.0

File: Simulation/Button/button.urdf (robot description, URDF)
Before this commit: robot Button_Assembly, 3 links, 2 joints
Links:
- link World: mass None -> 0.1412; geometry collision mesh filename=meshes/tn__corpo1_dC_Corpo1_Mesh.obj scale=1. 1. 1.; visual mesh filename=meshes/tn__corpo1_dC_Corpo1_Mesh.obj scale=1. 1. 1.
- link button_pivot: mass None -> 0.0377; geometry collision mesh filename=meshes/tn__botao1_dC_Corpo1_Mesh.obj scale=1. 1. 1.; visual mesh filename=meshes/tn__botao1_dC_Corpo1_Mesh.obj scale=1. 1. 1.
- link lid_pivot: mass None -> 0.0824; geometry collision mesh filename=meshes/tn__Tampa1_dC_Corpo1_Mesh.obj scale=1. 1. 1.; visual mesh filename=meshes/tn__Tampa1_dC_Corpo1_Mesh.obj scale=1. 1. 1.
Joints:
- joint PrismaticJoint: limit lower=-0.01 upper=0. effort=10000000. velocity=0. -> lower=-0.01 upper=0. effort=100.0 velocity=1.0
- joint RevoluteJoint: limit lower=-1.5707963 upper=0.6981317 effort=0. velocity=0. -> lower=-1.5707963 upper=0.6981317 effort=100.0 velocity=10.0

File: Simulation/Circuit Breaker/Circuit_Breaker_Assembly.urdf (robot description, URDF)
Before this commit: robot Circuit_Breaker_Assembly, 2 links, 1 joints
Links:
- link World: mass None -> 0.2636
- link lever_pivot: mass None -> 0.0264
Joints:
- joint RevoluteJoint: limit lower=-0.5235988 upper=0.5235988 effort=10000000. velocity=0. -> lower=-0.5235988 upper=0.5235988 effort=100.0 velocity=10.0

File: Simulation/Circuit Breaker/circuit_breaker.urdf (robot description, URDF)
Before this commit: robot Circuit_Breaker_Assembly, 3 links, 2 joints
Links:
- link World: mass None -> 0.0500
- link body_pivot: mass None -> 0.2636; geometry collision mesh filename=meshes/tn__corpo1_dC_Corpo1_Mesh.obj scale=1. 1. 1.; visual mesh filename=meshes/tn__corpo1_dC_Corpo1_Mesh.obj scale=1. 1. 1.
- link lever_pivot: mass None -> 0.0264; geometry collision mesh filename=meshes/tn__Alavanca1_zH_Corpo1_Mesh.obj scale=1. 1. 1.; visual mesh filename=meshes/tn__Alavanca1_zH_Corpo1_Mesh.obj scale=1. 1. 1.
Joints:
- joint RevoluteJoint: limit lower=-0.5235988 upper=0.5235988 effort=10000000. velocity=0. -> lower=-0.5235988 upper=0.5235988 effort=100.0 velocity=10.0

File: Simulation/Drawer/Drawer_Assembly.urdf (robot description, URDF)
Before this commit: robot Drawer_Assembly, 1 links, 0 joints
Links:
- link Drawer_Assembly: mass None -> 0.0050

File: Simulation/Honeycomb/Honeycomb.urdf (robot description, URDF)
Before this commit: robot Honeycomb, 1 links, 0 joints
Links:
- link Honeycomb: mass None -> 10.0000; geometry collision mesh filename=meshes/Mesh.obj scale=0.001000 0.001000 0.001000; visual mesh filename=meshes/Mesh.obj scale=0.001000 0.001000 0.001000

File: Simulation/Honeycomb/Honeycomb_Panel.urdf (robot description, URDF)
Before this commit: robot Honeycomb_Panel, 1 links, 0 joints
Links:
- link Honeycomb_Panel: mass None -> 0.0050

File: Simulation/Key/Key_assembly.urdf (robot description, URDF)
Before this commit: robot Key_assembly, 1 links, 0 joints
Links:
- link Key_assembly: mass None -> 0.0050

File: Simulation/Lamp/Lamp_Assembly.urdf (robot description, URDF)
Before this commit: robot Lamp_Assembly, 3 links, 2 joints
Links:
- link World: mass None -> 0.3005
- link lamp_pivot: mass None -> 0.0219
- link rotation_pivot: mass None -> 0.0500
Joints:
- joint PrismaticJoint: limit lower=0. upper=0.024 effort=10000000. velocity=0. -> lower=0. upper=0.024 effort=100.0 velocity=1.0

File: Simulation/Shock Absorber/Shock_Absorber_Assembly.urdf (robot description, URDF)
Before this commit: robot Shock_Absorber_Assembly, 1 links, 0 joints
Links:
- link Montagem_Principal: mass None -> 0.0050; geometry collision mesh filename=meshes/Corpo3.obj scale=0.001000 0.001000 0.001000; collision mesh filename=meshes/MeshInstance_1_Corpo1.obj scale=0.001000 0.001000 0.001000

File: Simulation/Threads/M14 Thread/M14.urdf (robot description, URDF)
Before this commit: robot M14, 3 links, 2 joints
Links:
- link World: mass None -> 0.3025
- link eixo_rot_porca: mass None -> 0.0050
- link eixo_trans_porca: mass None -> 0.0104
Joints:
- joint PrismaticJoint: limit lower=-0.005 upper=0.012 effort=10000000. velocity=0. -> lower=-0.005 upper=0.012 effort=100.0 velocity=1.0

File: Simulation/Threads/M8 Thread/M8_Assy.urdf (robot description, URDF)
Before this commit: robot M8_Assy, 3 links, 2 joints
Links:
- link World: mass None -> 0.3025
- link nut_pivot: mass None -> 0.0050
- link rot_pivot: mass None -> 0.0500
Joints:
- joint PrismaticJoint: limit lower=0. upper=0.015 effort=10000000. velocity=0. -> lower=0. upper=0.015 effort=100.0 velocity=1.0

File: Simulation/Valves/Gate Valve/Small Valve/Small_Valve.urdf (robot description, URDF)
Before this commit: robot Small_Valve, 3 links, 2 joints
Links:
- link eixo_trans: mass None -> 0.0050
- link pivot_registro: mass None -> 0.0050
- link valvula_gaveta: mass None -> 0.5310
Joints:
- joint PrismaticJoint: limit lower=-0.02 upper=0.015 effort=10000000. velocity=0. -> lower=-0.02 upper=0.015 effort=100.0 velocity=1.0

File: Simulation/Valves/Gate Valve/Small Valve/small_valve.urdf (robot description, URDF)
Before this commit: robot Small_Valve, 3 links, 2 joints
Links:
- link eixo_trans: mass None -> 0.0050; geometry collision mesh filename=./meshes/Mesh_22.obj scale=1. 1. 1.; visual mesh filename=./meshes/Mesh_21.obj scale=1. 1. 1.
- link pivot_registro: mass None -> 0.0050
- link valvula_gaveta: mass None -> 0.5310
Joints:
- joint PrismaticJoint: limit lower=-0.02 upper=0.015 effort=10000000. velocity=0. -> lower=-0.02 upper=0.015 effort=100.0 velocity=1.0

File: Simulation/Valves/Lever Valve/Ball Valve/Ball_Valve.urdf (robot description, URDF)
Before this commit: robot Ball_Valve, 2 links, 1 joints
Links:
- link alavanca_pivot: mass None -> 0.1230
- link valvula_esfera: mass None -> 0.2689
Joints:
- joint RevoluteJoint: limit lower=-1.5707963 upper=0. effort=10000000. velocity=0. -> lower=-1.5707963 upper=0. effort=100.0 velocity=10.0

File: Simulation/Valves/Lever Valve/Ball Valve/ball_valve.urdf (robot description, URDF)
Before this commit: robot Ball_Valve, 2 links, 1 joints
Links:
- link alavanca_pivot: mass None -> 0.1230; geometry collision mesh filename=meshes/Mesh_1.obj scale=1. 1. 1.; visual mesh filename=meshes/Mesh_1.obj scale=1. 1. 1.
- link valvula_esfera: mass None -> 0.2689; geometry collision mesh filename=meshes/Mesh.obj scale=1. 1. 1.; visual mesh filename=meshes/Mesh.obj scale=1. 1. 1.
Joints:
- joint RevoluteJoint: limit lower=-1.5707963 upper=0. effort=10000000. velocity=0. -> lower=-1.5707963 upper=0. effort=100.0 velocity=10.0
