Commit message: more urdfs

File: Simulation/Honeycomb/Honeycomb.urdf (robot description, URDF)
Before this commit: robot Honeycomb, 1 links, 0 joints
Links:
- link Honeycomb: geometry collision mesh filename=meshes/Mesh.obj scale=1. 1. 1.; visual mesh filename=meshes/Mesh.obj scale=1. 1. 1.

Commit message: Fixed inertia

File: Simulation/Honeycomb/Honeycomb.urdf (robot description, URDF)
Before this commit: robot Honeycomb, 1 links, 0 joints
Links:
- link Honeycomb: mass 10.0000 -> 0.1732; geometry collision mesh filename=meshes/Mesh.obj scale=0.001000 0.001000 0.001000; visual mesh filename=meshes/Mesh.obj scale=0.001000 0.001000 0.001000

File: Simulation/Valves/Lever Valve/Ball Valve/Ball_Valve_Friction_Ring_Set.urdf (robot description, URDF)
Before this commit: robot Ball_Valve_Friction_Ring_Set, 1 links, 0 joints
Links:
- link Ball_Valve_Friction_Ring_Set: mass 10.0000 -> 0.0050; geometry collision mesh filename=meshes/Corpo1_Mesh.obj scale=0.001000 0.001000 0.001000; collision mesh filename=meshes/Corpo2_Mesh.obj scale=0.001000 0.001000 0.001000
