Commit message: Stabilize lamp collision for PhysX grasping.
Replace CAD-shell convex hulls on lamp_pivot with two cylinders along
the bulb axis, and scale the link mass to 0.20 kg so grasp contacts
no longer explode.

File: Simulation/Lamp/Lamp_Assembly.urdf (robot description, URDF)
Before this commit: robot Lamp_Assembly, 3 links, 2 joints
Links:
- link lamp_pivot: mass 0.0219 -> 0.20; geometry collision cylinder length=0.030 radius=0.014; collision cylinder length=0.080 radius=0.028
