Commit message: Fix URDF articulation and collision geometry for M8, M30 and Peg Insertion
- M8 Thread (M8_Assy.urdf): Replace base mesh collider with primitive box and cylinders to prevent single-convex-hull cone approximation from blocking gripper contact. Increase nut mass to 20 g to stabilize GPU PhysX grasp contacts, and structure continuous RevoluteJoint + PrismaticJoint along +X.
- M30 Thread (M30.urdf): Align plate normal to +X consistent with the board and other mechanisms. Move prismatic joint to the nut (World -> rot_pivot -> Nut), and replace conical base mesh collider with box and cylinder primitives.
- Peg Insertion (Peg_Insertion.urdf, Peg_insertion_1..5.urdf): Free the peg from static FixedJoint welds into an articulated revolute and prismatic screw pair along +X. Replace plate collision with primitive box and adjust peg mass to 20 g for grasp stability. Add canonical Peg_Insertion.urdf and update hole configurations 1..5.

File: Simulation/Peg Insertion/Peg_Insertion.urdf (robot description, URDF)
Before this commit: robot Peg_insertion_4, 3 links, 2 joints
Joints:
- joint RevoluteJoint: origin xyz=0 -0.028569 0.014372 rpy=0 1.5707963 0 -> xyz=0 0 0 rpy=0 1.5707963 0

File: Simulation/Peg Insertion/Peg_insertion_1.urdf (robot description, URDF)
Before this commit: robot Peg_insertion_1, 2 links, 1 joints
Links:
- removed link Base
- added link peg, mass 0.02; collision mesh filename=meshes/Al__a_Corpo1.obj scale=1 1 1; visual mesh filename=meshes/Al__a_Corpo1.obj scale=1 1 1
- added link rot_pivot, mass 0.005
- link World: mass 0.0050 -> 0.1008; geometry collision box size=0.015 0.076 0.076; visual mesh filename=meshes/Base_principal_Corpo1.obj scale=1 1 1
Joints:
- removed joint FixedJoint
- added joint PrismaticJoint: type prismatic, parent rot_pivot, child peg, origin xyz=0 0 0 rpy=0 0 0, axis 0 0 1, limit lower=0.0 upper=0.020 effort=100.0 velocity=1.0
- added joint RevoluteJoint: type continuous, parent World, child rot_pivot, origin xyz=0 0 0 rpy=0 1.5707963 0, axis 0 0 1

File: Simulation/Peg Insertion/Peg_insertion_2.urdf (robot description, URDF)
Before this commit: robot Peg_insertion_2, 2 links, 1 joints
Links:
- removed link Base
- added link peg, mass 0.02; collision mesh filename=meshes/Al__a_Corpo1.obj scale=1 1 1; visual mesh filename=meshes/Al__a_Corpo1.obj scale=1 1 1
- added link rot_pivot, mass 0.005
- link World: mass 0.0050 -> 0.1008; geometry collision box size=0.015 0.076 0.076; visual mesh filename=meshes/Base_principal_Corpo1.obj scale=1 1 1
Joints:
- removed joint FixedJoint
- added joint PrismaticJoint: type prismatic, parent rot_pivot, child peg, origin xyz=0 0 0 rpy=0 0 0, axis 0 0 1, limit lower=0.0 upper=0.020 effort=100.0 velocity=1.0
- added joint RevoluteJoint: type continuous, parent World, child rot_pivot, origin xyz=0 0 0.034988 rpy=0 1.5707963 0, axis 0 0 1

File: Simulation/Peg Insertion/Peg_insertion_3.urdf (robot description, URDF)
Before this commit: robot Peg_insertion_3, 2 links, 1 joints
Links:
- removed link Base
- added link peg, mass 0.02; collision mesh filename=meshes/Al__a_Corpo1.obj scale=1 1 1; visual mesh filename=meshes/Al__a_Corpo1.obj scale=1 1 1
- added link rot_pivot, mass 0.005
- link World: mass 0.0050 -> 0.1008; geometry collision box size=0.015 0.076 0.076; visual mesh filename=meshes/Base_principal_Corpo1.obj scale=1 1 1
Joints:
- removed joint FixedJoint
- added joint PrismaticJoint: type prismatic, parent rot_pivot, child peg, origin xyz=0 0 0 rpy=0 0 0, axis 0 0 1, limit lower=0.0 upper=0.020 effort=100.0 velocity=1.0
- added joint RevoluteJoint: type continuous, parent World, child rot_pivot, origin xyz=0 -0.00015 -0.02495 rpy=0 1.5707963 0, axis 0 0 1

File: Simulation/Peg Insertion/Peg_insertion_5.urdf (robot description, URDF)
Before this commit: robot Peg_insertion_5, 2 links, 1 joints
Links:
- removed link Base
- added link peg, mass 0.02; collision mesh filename=meshes/Al__a_Corpo1.obj scale=1 1 1; visual mesh filename=meshes/Al__a_Corpo1.obj scale=1 1 1
- added link rot_pivot, mass 0.005
- link World: mass 0.0050 -> 0.1008; geometry collision box size=0.015 0.076 0.076; visual mesh filename=meshes/Base_principal_Corpo1.obj scale=1 1 1
Joints:
- removed joint FixedJoint
- added joint PrismaticJoint: type prismatic, parent rot_pivot, child peg, origin xyz=0 0 0 rpy=0 0 0, axis 0 0 1, limit lower=0.0 upper=0.020 effort=100.0 velocity=1.0
- added joint RevoluteJoint: type continuous, parent World, child rot_pivot, origin xyz=0 0.028087 0 rpy=0 1.5707963 0, axis 0 0 1

File: Simulation/Threads/M30 Thread/M30.urdf (robot description, URDF)
Before this commit: robot M30, 3 links, 2 joints
Links:
- removed link Base
- added link rot_pivot, mass 0.005
- link Nut: geometry collision mesh filename=meshes/Nut_Corpo1.obj scale=1 1 1; visual mesh filename=meshes/Nut_Corpo1.obj scale=1 1 1
- link World: mass 0.0500 -> 0.4369; geometry collision box size=0.015 0.076 0.076; collision cylinder length=0.050 radius=0.0150
Joints:
- joint PrismaticJoint: axis 0. 0. 1. -> 0 0 1; child Base -> Nut; limit lower=-0.05 upper=0. effort=100.0 velocity=1.0 -> lower=0.0 upper=0.025 effort=100.0 velocity=1.0; origin xyz=0. 0. 0. rpy=0. 0. 0. -> xyz=0 0 0 rpy=0 0 0; parent World -> rot_pivot
- joint RevoluteJoint: axis 0. 0. 1. -> 0 0 1; child Nut -> rot_pivot; origin xyz=0. 0. 0.015649 rpy=0. 0. 0. -> xyz=0.015649 0 0 rpy=0 1.5707963 0

File: Simulation/Threads/M8 Thread/M8_Assy.urdf (robot description, URDF)
Before this commit: robot M8_Assy, 3 links, 2 joints
Links:
- link World: geometry collision box size=0.015 0.076 0.076; collision cylinder length=0.0104 radius=0.0053
- link nut_pivot: mass 0.0050 -> 0.02; geometry collision mesh filename=meshes/M8_Nut_Corpo1_Mesh.obj scale=1 1 1; visual mesh filename=meshes/M8_Nut_Corpo1_Mesh.obj scale=1 1 1
- link rot_pivot: mass 0.0500 -> 0.005; geometry 
Joints:
- joint PrismaticJoint: axis 1. 0. 0. -> 1 0 0; limit lower=0. upper=0.015 effort=100.0 velocity=1.0 -> lower=0.0 upper=0.015 effort=100.0 velocity=1.0; origin xyz=0. 0. 0. rpy=0. 0. 0. -> xyz=0 0 0 rpy=0 0 0
- joint RevoluteJoint: axis 1. 0. 0. -> 1 0 0; origin xyz=0. 0. 0. rpy=0. 0. 0. -> xyz=0 0 0 rpy=0 0 0
